File: usbtherm-kicad/usbtherm.kicad_sch (KiCad schematic)
At the start: 19 parts, among them CON1 USB-A PLUG, J1 ISP, U1 ATtiny85-20S, U2 TMP36, U3 HIH-5030-001

Commit message: add PCB
Parts:
- removed C1: 100nF, Capacitor_SMD:C_1812_4532Metric_Pad1.57x3.40mm_HandSolder, symbol Device:C
- removed J1: ISP, symbol Connector:Conn_01x06_Female
- added J1: ISP, Connector_PinSocket_2.54mm:PinSocket_1x05_P2.54mm_Vertical, symbol Connector:Conn_01x05_Female
Connections:
- net +5V: now reaches C2.1, C3.2, CON1.1 (VBUS), R3.1, R6.2, U1.8 (VCC), U2.2 (+VS), U2.4 (~{SHUTDOWN}), U3.3 (+VE)
- net +5V: now also J1.2 (VCC)
- net at R2.1, U1.7 (PB2): now also J1.3 (SCK)
- net at R5.2, U1.5 (AREF/PB0): now also J1.4 (MOSI)
- net at R1.1, U1.6 (PB1): now also J1.1 (MISO)
- net at U1.1 (~{RESET}/PB5): now also J1.5 (RESET)
